File: 70mm by 50mm Ver2.4 ATmega328p/Solder-Reflow-Plate.kicad_sch (KiCad schematic)
At the start: 35 parts

Commit message: Added: PCB FIle
Parts:
- renumbered 12V to 12V1, 5V to 5V1, C10 to C1, C3 to C10, C14 to C11, C4 to C12, C19 to C13, C5 to C14, C6 to C15, C7 to C16, C9 to C17, C12 to C2, C13 to C3, C2 to C4, C16 to C5, C17 to C6, C1 to C7, C18 to C8, C15 to C9, D3 to D2, D2 to D3, DNSW to DNSW1, ICSP to ICSP1, MOSFET to MOSFET1, OLED to OLED1, R5 to R1, R1 to R2, R2 to R3, R6 to R4, R7 to R5, R4 to R6, TEMP to TEMP1, UC to UC1, UPSW to UPSW1
Connections:
- net 0V: no longer 12V1.2, 12V1.3, 5V1.1 (ADJ(GND)), C10.1, C11.1, C12.2, C13.1, C14.1, C15.2, C17.2, C4.2, C5.1, C6.1, C7.1, C8.1, D1.1, ICSP1.6, MOSFET1.3 (S), OLED1.4 (GND), R1.2, R3.1, R4.2, R6.1, TEMP1.3 (GND), UC1.21 (GND)
- new net GND: 12V1.2, 12V1.3, 5V1.1 (ADJ(GND)), C10.1, C11.1, C12.2, C13.1, C14.1, C15.2, C17.2, C4.2, C5.1, C6.1, C7.1, C8.1, D1.1, ICSP1.6, MOSFET1.3 (S), OLED1.4 (GND), R1.2, R3.1, R4.2, R6.1, TEMP1.3 (GND), UC1.21 (GND)
